File: STM32F10xPill_GPS_Locator/STM32F10xPill_GPS_Locator.kicad_sch (KiCad schematic)
At the start: 0 parts

Commit message: Add controller and clocks
Other:
- note added: "Controller"
- note added: "Peripherals"
- note added: "Power Supply"
- company: (none) -> MTP
- title: (none) -> STM32F100C4T6B GPS Locator
Changed lines of the file:
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@@
 	(generator "eeschema")
 	(generator_version "9.0")
-	(paper "A4")
+	(paper "A3")
+	(title_block
+		(title "STM32F100C4T6B GPS Locator")
+		(date "2025-03-06")
+		(rev "1.0.0")
+		(company "MTP")
+	)
 	(text "STM32F100C4T6B Handheld GPS Locator"
 		(exclude_from_sim no)
-		(at 147.066 26.162 0)
-		(effects
-			(font
-				(size 5.08 5.08)
+		(at 212.598 31.242 0)
+		(effects
+			(font
+				(size 12.7 12.7)
 				(thickness 0.381)
 				(bold yes)
@@
 		)
 	)
+	(text "Peripherals"
+		(exclude_from_sim no)
+		(at 323.342 104.648 0)
+		(effects
+			(font
+				(size 7.62 7.62)
+				(thickness 0.3175)
+			)
+		)
+	)
+	(text "Controller"
+		(exclude_from_sim no)
+		(at 200.66 105.918 0)
+		(effects
+			(font
+				(size 7.62 7.62)
+				(thickness 0.3175)
+			)
+		)
+	)
 	(text "System Architecture"
 		(exclude_from_sim no)
-		(at 147.32 66.548 0)
-		(effects
-			(font
-				(size 2.794 2.794)
-				(thickness 0.3175)
-			)
+		(at 212.09 71.374 0)
+		(effects
+			(font
+				(size 7.62 7.62)
+				(thickness 0.3175)
+			)
+		)
+	)
+	(text "Power Supply"
+		(exclude_from_sim no)
+		(at 87.63 104.648 0)
+		(effects
+			(font
+				(size 7.62 7.62)
+				(thickness 0.3175)
+			)
+		)
+	)
+	(text_box "DESIGN NOTE:\nExample text for debug notes."
+		(exclude_from_sim no)
+		(at 91.44 257.81 0)
+		(size 30.48 20.32)
+		(margins 2 2 2 2)
+		(stroke
+			(width 1)
+			(type solid)
+			(color 255 165 0 1)
+		)
+		(fill
+			(type none)
+		)
+		(effects
+			(font
+				(face "Arial")
+				(size 2 2)
+				(color 0 0 0 1)
+			)
+			(justify left top)
+		)
+	)
+	(text_box "DESIGN NOTE:\nExample text for cautionary design notes."
+		(exclude_from_sim no)
+		(at 126.365 257.81 0)
+		(size 30.48 20.32)
+		(margins 2 2 2 2)
+		(stroke
+			(width 1)
+			(type solid)
+			(color 250 236 0 1)
+		)
+		(fill
+			(type none)
+		)
+		(effects
+			(font
+				(face "Arial")
+				(size 2 2)
+				(color 0 0 0 1)
+			)
+			(justify left top)
+		)
+	)
+	(text_box "DESIGN NOTE:\nExample text for critical design notes."
+		(exclude_from_sim no)
+		(at 161.29 257.81 0)
+		(size 30.48 20.32)
+		(margins 2.25 2.25 2.25 2.25)
+		(stroke
+			(width 1.5)
+			(type solid)
+			(color 255 0 0 1)
+		)
+		(fill
+			(type none)
+		)
+		(effects
+			(font
+				(face "Arial")
+				(size 2 2)
+				(thickness 0.4)
+				(bold yes)
+				(color 255 0 0 1)
+			)
+			(justify left top)
+		)
+	)
+	(text_box "DESIGN NOTE:\nExample text for informational design notes."
+		(exclude_from_sim no)
+		(at 56.515 257.81 0)
+		(size 30.48 20.32)
+		(margins 2 2 2 2)
+		(stroke
+			(width 1)
+			(type solid)
+			(color 200 200 200 1)
+		)
+		(fill
+			(type none)
+		)
+		(effects
+			(font
+				(face "Arial")
+				(size 2 2)
+				(color 0 0 0 1)
+			)
+			(justify left top)
+		)
+	)
+	(text_box "LAYOUT NOTE:\nExample text for critical layout guidelines."
+		(exclude_from_sim no)
+		(at 196.215 257.81 0)
+		(size 30.48 20.32)
+		(margins 2.25 2.25 2.25 2.25)
+		(stroke
+			(width 1.5)
+			(type solid)
+			(color 0 0 255 1)
+		)
+		(fill
+			(type none)
+		)
+		(effects
+			(font
+				(face "Arial")
+				(size 2 2)
+				(thickness 0.4)
+				(bold yes)
+				(color 0 0 255 1)
+			)
+			(justify left top)
 		)
 	)
 	(sheet
-		(at 91.44 78.74)
-		(size 31.75 24.13)
+		(at 52.07 116.84)
+		(size 68.58 66.04)
 		(exclude_from_sim no)
 		(in_bom yes)
@@
 		)
 		(property "Sheetname" "Power Supply"
-			(at 91.44 78.0284 0)
+			(at 52.07 116.1284 0)
 			(effects
 				(font
@@
 		)
 		(property "Sheetfile" "Power Supply.kicad_sch"
-			(at 91.44 103.4546 0)
+			(at 52.07 183.4646 0)
 			(effects
 				(font
@@
 	)
 	(sheet
-		(at 128.27 91.44)
-		(size 31.75 24.13)
+		(at 167.64 116.84)
+		(size 68.58 66.04)
 		(exclude_from_sim no)
 		(in_bom yes)
@@
 		)
 		(property "Sheetname" "Controller"
-			(at 128.27 90.7284 0)
+			(at 167.64 116.1284 0)
 			(effects
 				(font
@@
 		)
 		(property "Sheetfile" "Controller.kicad_sch"
-			(at 128.27 116.1546 0)
+			(at 167.64 183.4646 0)
 			(effects
 				(font
@@
 	)
 	(sheet
-		(at 165.1 78.74)
-		(size 31.75 24.13)
+		(at 290.83 118.11)
+		(size 68.58 66.04)
 		(exclude_from_sim no)
 		(in_bom yes)
@@
 		)
 		(property "Sheetname" "Peripherals"
-			(at 165.1 78.0284 0)
+			(at 290.83 117.3984 0)
 			(effects
 				(font
@@
 		)
 		(property "Sheetfile" "Peripherals.kicad_sch"
-			(at 165.1 103.4546 0)
-			(effects
-				(font
+			(at 290.83 184.7346 0)
+			(effects
+				(font
