File: STM32F10xPill_GPS_Locator/Power Supply.kicad_sch (KiCad schematic)
At the start: 0 parts

Commit message: Add controller and clocks
Other:
- company: (none) -> MTP
- title: (none) -> STM32F100C4T6B GPS Locator
Changed lines of the file:
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@@
 	(generator "eeschema")
 	(generator_version "9.0")
-	(paper "A4")
+	(paper "A3")
+	(title_block
+		(title "STM32F100C4T6B GPS Locator")
+		(date "2025-03-06")
+		(rev "1.0.0")
+		(company "MTP")
+	)
 )
