File: STM32F10xPill_GPS_Locator/STM32F10xPill_GPS_Locator.kicad_pcb (KiCad board)
At the start: 2 copper layers, 70 x 91 mm, 111 parts, among them J1 Conn_01x03, J2 Conn_01x05, J3 Conn_01x02, J4 734120110, Q1 2301D, SW2 TS-1092S-B3D2-G, SW3 TS-1092S-B3D2-G, SW4 Power, SW5 TS-1092S-B3D2-G, SW6 PTS645VH58-2 LFS, U1 STM32F100C4T6, U2 MCP73871T-2CCI/ML, U3 TPS61022, U5 QMC5883P, U6 AT2659S, U7 ATGM336H-5N31, Y1 16MHz, Y2 32.768kHz

Commit message: Initial placement completed
Parts:
- removed the C23 at (328.1, 46.8)
- added G***: LOGO, LOGO, B.Cu at (126.0, 109.5)
- added REF**: MTP Logo 5mm Low Detail Copper, Watermarks:MTP Logo 5mm Low Detail Copper, F.Cu at (126.0, 137.5)
- added REF**: michaelpate.net QR Code 10mm, Watermarks:michaelpate.net QR Code 10mm, B.Cu at (125.1, 125.0)
- added REF**: MTP Logo 10mm Low Detail Copper, Watermarks:MTP Logo 10mm Low Detail Copper, B.Cu at (180.5, 129.5)
- U3: value TPS61022 -> TPS61022RWUR; footprint Package_TO_SOT_SMD:SC-74A-5_1.55x2.9mm_P0.95mm -> Package_DFN_QFN:Texas_RWU0007A_VQFN-7_2x2mm_P0.5mm
- moved L1 219.7 mm to (141.4, 131.1), turned to -90 degrees
- moved C18 217.6 mm to (136.4, 131.1), turned to 90 degrees
- moved C23 215.0 mm to (127.2, 54.9), turned to -90 degrees
- moved C19 213.2 mm to (137.4, 128.6), turned to 180 degrees
- moved R19 212.8 mm to (135.3, 131.1), turned to 90 degrees
- moved R20 211.7 mm to (136.4, 133.6), turned to 90 degrees
- moved U3 209.4 mm to (138.4, 131.1), turned to -90 degrees
- moved U5 209.2 mm to (130.4, 56.6), turned to 180 degrees
- moved JP3 208.3 mm to (136.9, 58.6), turned to 90 degrees
- moved NT2 207.5 mm to (145.9, 132.1), turned to 180 degrees
- moved NT4 206.5 mm to (124.9, 127.1), turned to 180 degrees
- moved C22 204.9 mm to (133.2, 54.9), turned to -90 degrees
- moved TP9 203.9 mm to (134.4, 133.6)
- moved C17 203.9 mm to (148.4, 133.0), turned to 90 degrees
- moved TP10 203.3 mm to (134.9, 127.1)
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- renumbered C27 to C13, C13 to C14, C14 to C15, C15 to C16, C16 to C17, C17 to C18, C18 to C19, C19 to C20, C20 to C21, C21 to C22, C22 to C23, C23 to C24, C24 to C25, C25 to C26, C26 to C27, R9 to R10, R10 to R11, R11 to R12, R12 to R13, R13 to R14, R14 to R15, R15 to R16, R16 to R17, R17 to R18, R18 to R19, R19 to R20, R20 to R21, R21 to R22, R22 to R23, R23 to R24, R24 to R9, SW6 to SW1, TP14 to TP10, TP15 to TP11, TP16 to TP12, TP17 to TP13, TP18 to TP14, TP19 to TP15, TP20 to TP16, TP8 to TP4, TP9 to TP5, TP10 to TP6, TP11 to TP7, TP12 to TP8, TP13 to TP9
Connections:
- U6 pad 5: +3.3V -> /Peripherals/LNA_VCC
Other:
- board text added: "+++"
- board text added: "+3.3v"
- board text added: "---"
- board text added: "1"
- board text added: "3v3"
- board text added: "5V IN"
- board text added: "5V Input"
- board text added: "8"
- board text added: "<-- Battery Positive"
- board text added: "A"
- board text added: "B"
- board text added: "BATT CHARGE"
- board text added: "BATT LOW"
- board text added: "BL"
- board text added: "BOOT0"
- board text added: "Battery Positive -->"
- board text added: "Bootloader"
- board text added: "C"
- board text added: "CE"
- board text added: "CLK"
- board text added: "Cache me if you can!"
- board text added: "Cache-Master F1"
- board text added: "Clock"
- board text added: "DC"
- board text added: "Data"
- board text added: "Designed by Michael Pate v1.0 03/2025"
- board text added: "GND"
- board text added: "GPS 1PPS"
- board text added: "GPS BATT"
- board text added: "GPS ON/OFF"
- board text added: "GPS VCC"
- board text added: "JLCJLCJLC"
- board text added: "LCD BACKLIGHT"
- board text added: "LCD Header"
- board text added: "LNA VCC"
- board text added: "MCU VDD"
- board text added: "MOSI"
- board text added: "Normal"
- board text added: "OFF"
- board text added: "ON"
- board text added: "PC13"
- board text added: "PWR SW"
- board text added: "Power Switch"
- board text added: "QMC VCC"
- board text added: "RESET"
- board text added: "RST"
- board text added: "Reset"
- board text added: "SWD PROG."
- board text added: "SWD. Program"
- board text added: "VCC"
- board text added: "geocaching.com"
- board text added: "michaelpate.net"
